File: hardware/kicad/cropdroid-room/cropdroid-room.kicad_pcb (KiCad board)
At the start: 2 copper layers, 273.1 x 110.5 mm, 43 parts, among them CON1 SJ1-3523N, CON2 SJ1-3523N, CON3 SJ1-3523N, CON4 SJ1-3523N, J1 OSTTC020162, J2 PJ-102A, J3 OSTTC020162, J4 OSTTC020162, J5 OSTTC020162, J6 OSTTC020162, J7 640456-3, J8 640456-3, J9 640456-3, K1 T9AS1D12-15, K2 T9AS1D12-15, K3 T9AS1D12-15, K4 T9AS1D12-15, K5 T9AS1D12-15, Q1 ULN2003AN, U1 PPTC151LFBN-RC, U2 PPTC151LFBN-RC

Commit message: finalize prototype v0.1a
Other:
- board text added: "Channel 0"
- board text added: "Channel 1"
- board text added: "Channel 2"
- board text added: "Channel 3"
- board text added: "Channel 4"
- board text added: "DHT22 Bottom"
- board text added: "DHT22 Canopy"
- board text added: "DHT22 Top"
- board text removed: "A/C"
- board text removed: "Dehumidifier"
- board text removed: "Heater"
- board text removed: "Lighting"
- board text removed: "Ventilation"
Changed lines of the file:
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@@
   (general
     (thickness 1.6)
-    (drawings 14)
+    (drawings 17)
     (tracks 286)
     (zones 0)
@@
   (module T9AS1D12-15:RELAY_T9AS1D12-15 (layer F.Cu)
     (at 229.362 53.594)
-    (fp_text reference K4 (at -3.665025 -27.220035) (layer F.SilkS)
+    (fp_text reference K4 (at -7.112 -26.924) (layer F.SilkS)
       (effects (font (size 1.395488 1.395488) (thickness 0.015)))
     )
@@
       (effects (font (size 0.787402 0.787402) (thickness 0.015)))
     )
-    (fp_text user PPTC151LFBN-RC (at 10.7785 3.81654) (layer F.SilkS)
+    (fp_text user PPTC151LFBN-RC (at 5.588 3.048) (layer F.SilkS)
       (effects (font (size 1.001717 1.001717) (thickness 0.015)))
     )
@@
       (effects (font (size 0.787402 0.787402) (thickness 0.015)))
     )
-    (fp_text user PPTC151LFBN-RC (at 10.7785 3.81654) (layer F.SilkS)
+    (fp_text user PPTC151LFBN-RC (at 5.588 -3.048) (layer F.SilkS)
       (effects (font (size 1.001717 1.001717) (thickness 0.015)))
     )
@@
   (module T9AS1D12-15:RELAY_T9AS1D12-15 (layer F.Cu)
     (at 262.382 53.594)
-    (fp_text reference K5 (at -3.665025 -27.220035) (layer F.SilkS)
+    (fp_text reference K5 (at -7.112 -26.924) (layer F.SilkS)
       (effects (font (size 1.395488 1.395488) (thickness 0.015)))
     )
@@
   (module T9AS1D12-15:RELAY_T9AS1D12-15 (layer F.Cu)
     (at 196.342 53.594)
-    (fp_text reference K3 (at -3.665025 -27.220035) (layer F.SilkS)
+    (fp_text reference K3 (at -7.112 -26.924) (layer F.SilkS)
       (effects (font (size 1.395488 1.395488) (thickness 0.015)))
     )
@@
   (module T9AS1D12-15:RELAY_T9AS1D12-15 (layer F.Cu)
     (at 163.322 53.594)
-    (fp_text reference K2 (at -3.665025 -27.220035) (layer F.SilkS)
+    (fp_text reference K2 (at -7.112 -26.924) (layer F.SilkS)
       (effects (font (size 1.395488 1.395488) (thickness 0.015)))
     )
@@
   (module T9AS1D12-15:RELAY_T9AS1D12-15 (layer F.Cu)
     (at 130.302 53.594)
-    (fp_text reference K1 (at -3.665025 -27.220035) (layer F.SilkS)
+    (fp_text reference K1 (at -6.858 -26.924) (layer F.SilkS)
       (effects (font (size 1.395488 1.395488) (thickness 0.015)))
     )
@@
       (net 53 "Net-(CON1-Pad3)"))
   )
-  (gr_text Ventilation (at 266.954 65.024) (layer F.SilkS)
+  (gr_text "DHT22\nBottom" (at 241.554 88.138) (layer F.SilkS)
     (effects (font (size 1 1) (thickness 0.15)))
   )
-  (gr_text Dehumidifier (at 233.934 65.024) (layer F.SilkS)
+  (gr_text "DHT22\nCanopy" (at 208.28 87.63) (layer F.SilkS)
     (effects (font (size 1 1) (thickness 0.15)))
   )
-  (gr_text Heater (at 201.168 65.024) (layer F.SilkS)
+  (gr_text "DHT22\nTop" (at 174.498 87.63) (layer F.SilkS)
     (effects (font (size 1 1) (thickness 0.15)))
   )
-  (gr_text A/C (at 168.656 65.024) (layer F.SilkS)
+  (gr_text "Channel 4" (at 267.208 65.278) (layer F.SilkS)
     (effects (font (size 1 1) (thickness 0.15)))
   )
-  (gr_text Lighting (at 134.62 65.278) (layer F.SilkS)
+  (gr_text "Channel 3" (at 234.442 65.024) (layer F.SilkS)
     (effects (font (size 1 1) (thickness 0.15)))
   )
+  (gr_text "Channel 2" (at 201.168 65.278) (layer F.SilkS)
+    (effects (font (size 1 1) (thickness 0.15)))
+  )
+  (gr_text "Channel 1" (at 168.656 65.278) (layer F.SilkS)
+    (effects (font (size 1 1) (thickness 0.15)))
+  )
+  (gr_text "Channel 0" (at 135.382 65.278) (layer F.SilkS)
+    (effects (font (size 1 1) (thickness 0.15)))
+  )

Commit message: upgrade hardware to v0.2a (120v)
Parts:
- removed J3, J5: OSTTC020162, digikey-footprints:Term_Block_1x2_P5mm
- removed J7, J9: 640456-3, digikey-footprints:PinHeader_1x3_P2.54_Drill1.1mm
- added CON5: SJ1-3523N, digikey-footprints:Headphone_Jack_3.5mm_SJ1-3523N, F.Cu at (185.3, 132.8)
- added CON6: SJ1-3523N, digikey-footprints:Headphone_Jack_3.5mm_SJ1-3523N, F.Cu at (201.0, 133.0)
- added CON7: SJ1-3523N, digikey-footprints:Headphone_Jack_3.5mm_SJ1-3523N, F.Cu at (216.5, 132.8)
- added J10: 3-213598-2, 3-213598-2:TE_3-213598-2, F.Cu at (269.9, 26.7)
- added Screw: Drill, drill-hole:Drill_Hole, F.Cu at (312.4, 57.1)
- added Screw: Drill, drill-hole:Drill_Hole, F.Cu at (348.1, 134.6)
- added Screw: Drill, drill-hole:Drill_Hole, F.Cu at (50.8, 114.3)
- added Screw: Drill, drill-hole:Drill_Hole, F.Cu at (21.8, 21.8)
- added U3: PPTC151LFBN-RC, PPTC151LFBN-RC:PPTC151LFBN-RC, F.Cu at (106.8, 63.2)
- J1: value OSTTC020162 -> 703W-00_52; footprint digikey-footprints:Term_Block_1x2_P5mm -> 703W-00_52:52
- J2: value PJ-102A -> 3-213598-2; footprint digikey-footprints:Barrel_Jack_5.5mmODx2.1mmID_PJ-102A -> 3-213598-2:TE_3-213598-2
- J4, J6: value OSTTC020162 -> 3-213598-2; footprint digikey-footprints:Term_Block_1x2_P5mm -> 3-213598-2:TE_3-213598-2
- J8: value 640456-3 -> 3-213598-2; footprint digikey-footprints:PinHeader_1x3_P2.54_Drill1.1mm -> 3-213598-2:TE_3-213598-2
- U1: value PPTC151LFBN-RC -> IRM-30-12; footprint PPTC151LFBN-RC:PPTC151LFBN-RC -> IRM-30-12:IRM-30-12
- moved J1 203.0 mm to (339.7, 45.2), turned to 90 degrees
- moved U1 199.2 mm to (300.6, 71.0), turned to 270 degrees
- moved J2 120.9 mm to (137.8, 26.7), turned to 0 degrees
- moved J8 72.2 mm to (236.9, 26.7)
- moved J6 65.9 mm to (204.0, 26.7), turned to 0 degrees
- moved J4 34.2 mm to (170.8, 26.7), turned to 0 degrees
- moved R8 33.6 mm to (180.2, 122.9)
- moved R10 33.0 mm to (211.3, 122.9)
- moved CON2 28.6 mm to (237.2, 132.8)
- moved CON1 28.1 mm to (164.7, 132.8)
- moved R6 28.1 mm to (154.8, 132.1)
- moved R9 27.9 mm to (196.0, 122.9)
- moved G*** 24.1 mm to (28.2, 129.3)
- moved CON3 22.6 mm to (257.9, 132.8)
- moved CON4 22.6 mm to (273.4, 132.8)
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Connections:
- D1 pad 1: +12V -> Net-(D1-Pad1)
- D10 pad 2: +12V -> Net-(D10-Pad2)
- D2 pad 2: +12V -> Net-(D1-Pad1)
- D3 pad 1: +12V -> Net-(D3-Pad1)
- D4 pad 2: +12V -> Net-(D3-Pad1)
- D5 pad 1: +12V -> Net-(D5-Pad1)
- D6 pad 2: +12V -> Net-(D5-Pad1)
- D7 pad 1: +12V -> Net-(D7-Pad1)
- D8 pad 2: +12V -> Net-(D7-Pad1)
- D9 pad 1: +12V -> Net-(D10-Pad2)
- J2 pad 1: +12V -> Net-(J1-Pad3)
- J2 pad 2: GND -> Net-(J2-Pad2)
- J2 pad 3: Net-(J2-Pad3) -> Net-(J1-Pad2)
- J4 pad 1: Net-(J4-Pad1) -> Net-(J1-Pad3)
- J6 pad 1: Net-(J6-Pad1) -> Net-(J1-Pad3)
- J8 pad 1: Net-(CON1-Pad3) -> Net-(J1-Pad3)
- J8 pad 3: GND -> Net-(J1-Pad2)
- K1 pad 2: +12V -> Net-(D1-Pad1)
- K1 pad 3: Net-(J1-Pad2) -> Net-(J1-Pad1)
- K1 pad 4: Net-(J1-Pad1) -> Net-(J2-Pad2)
- K2 pad 2: +12V -> Net-(D3-Pad1)
- K2 pad 3: Net-(J3-Pad2) -> Net-(J1-Pad1)
- K2 pad 4: Net-(J3-Pad1) -> Net-(J4-Pad2)
- K3 pad 2: +12V -> Net-(D5-Pad1)
- K3 pad 3: Net-(J4-Pad2) -> Net-(J1-Pad1)
- K3 pad 4: Net-(J4-Pad1) -> Net-(J6-Pad2)
- K4 pad 2: +12V -> Net-(D7-Pad1)
- K4 pad 3: Net-(J5-Pad2) -> Net-(J1-Pad1)
- K4 pad 4: Net-(J5-Pad1) -> Net-(J8-Pad2)
- K5 pad 2: +12V -> Net-(D10-Pad2)
- K5 pad 3: Net-(J6-Pad2) -> Net-(J1-Pad1)
- K5 pad 4: Net-(J6-Pad1) -> Net-(J10-Pad2)
- Q1 pad 9: +12V -> Net-(Q1-Pad9)
- R10 pad 2: Net-(J9-Pad2) -> Net-(CON7-Pad2)
- R8 pad 2: Net-(J7-Pad2) -> Net-(CON5-Pad2)
- R9 pad 2: Net-(J8-Pad2) -> Net-(CON6-Pad2)
- U2 pad P$1: +12V -> Net-(U2-PadP$1)
- U2 pad P$10: Net-(CON4-Pad2) -> Net-(Q1-Pad4)
- U2 pad P$11: Net-(CON3-Pad2) -> Net-(Q1-Pad5)
- U2 pad P$12: Net-(CON2-Pad2) -> Net-(Q1-Pad6)
- U2 pad P$2: GND -> Net-(U2-PadP$2)
- U2 pad P$4: Net-(CON1-Pad3) -> GND
- U2 pad P$5: Net-(U2-PadP$5) -> Net-(CON1-Pad2)
- U2 pad P$6: Net-(Q1-Pad7) -> Net-(CON5-Pad2)
- U2 pad P$7: Net-(J9-Pad2) -> Net-(Q1-Pad1)
- U2 pad P$8: Net-(J8-Pad2) -> Net-(Q1-Pad2)
- U2 pad P$9: Net-(D11-Pad1) -> Net-(Q1-Pad3)
Routing:
- net +12V: track 473.4 -> 0.00 mm
- net Net-(J1-Pad1): track 21.5 -> 419.9 mm
- net Net-(Q1-Pad9): track 0.00 -> 391.7 mm
- net Net-(J1-Pad3): track 0.00 -> 303.3 mm
- net Net-(CON5-Pad2): track 0.00 -> 255.1 mm
- net Net-(J9-Pad2): track 248.5 -> 0.00 mm
- net Net-(CON7-Pad2): track 0.00 -> 241.1 mm
- net Net-(CON6-Pad2): track 0.00 -> 234.7 mm
- net Net-(J1-Pad2): track 25.6 -> 258.2 mm
- net Net-(J7-Pad2): track 225.4 -> 0.00 mm
- net Net-(J8-Pad2): track 222.9 -> 36.6 mm
- net Net-(D1-Pad1): track 0.00 -> 36.9 mm
- net Net-(J2-Pad2): track 0.00 -> 36.6 mm
- net Net-(J10-Pad2): track 0.00 -> 36.4 mm
- net Net-(D5-Pad1): track 0.00 -> 36.3 mm
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Other:
- board size 273.1 x 110.5 mm -> 342.9 x 132.1 mm
- net class Mains AC added: clearance 3.048, trace_width 5.08, via_dia 2.032, via_drill 0.381
- board text added: "CropDroid Room Controller CopyRight (c) Automate The Things, LLC Prototype v0.2a"
- board text removed: "CropDroid Room Controller CopyRight (c) Automate The Things, LLC Prototype v0.1a"

Commit message: final kicad v0.2a
Parts:
- moved Screw 31.2 mm to (22.1, 101.9)
- moved J2 12.8 mm to (150.5, 25.2)
- moved J4 12.8 mm to (216.7, 25.2)
- moved J5 12.8 mm to (249.6, 25.2)
- moved J3 12.8 mm to (183.5, 25.2)
- moved J6 12.8 mm to (282.6, 25.2)
- moved U1 12.7 mm to (313.3, 71.2)
- moved CON1 12.7 mm to (177.4, 133.1)
- moved CON2 12.7 mm to (249.9, 133.1)
- moved CON5 12.7 mm to (213.7, 133.2)
- moved CON7 12.7 mm to (229.2, 133.1)
- moved D1 12.7 mm to (133.2, 86.6)
- moved D2 12.7 mm to (141.9, 94.2)
- moved D5 12.7 mm to (199.3, 86.6)
- moved K3 12.7 mm to (209.2, 76.5)
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- renumbered CON5 to CON3, CON3 to CON4, CON6 to CON5, CON4 to CON6, J4 to J3, J6 to J4, J8 to J5, J10 to J6
Routing:
- net Net-(J1-Pad2): track 258.2 -> 243.3 mm
- net Net-(CON1-Pad2): track 245.2 -> 259.8 mm
- net Net-(D1-Pad2): track 92.6 -> 105.8 mm
- net Net-(CON3-Pad2): track 255.1 -> 268.2 mm
- net Net-(D5-Pad2): track 157.8 -> 170.8 mm
- net Net-(D9-Pad2): track 223.1 -> 236.0 mm
- net Net-(CON2-Pad2): track 281.7 -> 294.5 mm
- net Net-(CON5-Pad2): track 234.7 -> 247.5 mm
- net Net-(D7-Pad2): track 190.6 -> 203.4 mm
- net Net-(D3-Pad2): track 126.6 -> 139.4 mm
- net Net-(CON7-Pad2): track 241.1 -> 253.8 mm
- net Net-(CON6-Pad2): track 262.2 -> 274.9 mm
- net Net-(CON4-Pad2): track 270.3 -> 283.1 mm
- net Net-(D11-Pad1): track 68.0 -> 80.5 mm
- net Net-(CON1-Pad3): track 417.0 -> 422.5 mm
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Other:
- board size 342.9 x 132.1 mm -> 355.6 x 131.1 mm
