File: hardware/kicad/cropdroid-room-v3/cropdroid-room.kicad_pcb (KiCad board)
At the start: 2 copper layers, 377.2 x 131.1 mm, 62 parts, among them CON1 SJ1-3523N, CON2 SJ1-3523N, CON3 SJ1-3523N, CON4 SJ1-3523N, CON5 SJ1-3523N, CON6 SJ1-3523N, CON7 SJ1-3523N, J1 703W-00_52, J2 3-213598-2, J3 3-213598-2, J4 3-213598-2, J5 3-213598-2, J6 3-213598-2, J7 3-213598-2, K1 T9AS1D12-15, K2 T9AS1D12-15, K3 T9AS1D12-15, K4 T9AS1D12-15, K5 T9AS1D12-15, K6 T9AS1D12-15, Q1 ULN2003AN, U1 IRM-30-12, U2 PPTC151LFBN-RC, U3 PPTC151LFBN-RC

Commit message: fix kicad v0.3a co2 circuit missing diode and connection to microcontroller
Parts:
- added D15: 1N4001, Diode_THT:D_DO-41_SOD81_P10.16mm_Horizontal, F.Cu at (253.0, 157.0)
- renumbered D15 to D16, D16 to D17, D17 to D18, D18 to D19, D19 to D20, D20 to D21, D21 to D22, D22 to D23
Connections:
- Screw pad 1: (no net) -> GND (x4)
Routing:
- net Net-(D15-Pad1): track 0.00 -> 163.5 mm
- net Net-(CON2-Pad2): track 0.00 -> 9.94 mm
- net Net-(D6-Pad2): track 110.3 -> 112.7 mm
- net Net-(D22-Pad1): track 205.4 -> 203.1 mm
- net Net-(D20-Pad1): track 186.6 -> 185.4 mm

Commit message: more v0.3a fixes
Parts:
- D1: value 1N4001 -> 1N5400; footprint Diode_THT:D_DO-41_SOD81_P10.16mm_Horizontal -> Diode_THT:D_DO-201AD_P15.24mm_Horizontal
- D16: value 1N5400 -> 1N4001; footprint Diode_THT:D_DO-201AD_P15.24mm_Horizontal -> Diode_THT:D_DO-41_SOD81_P10.16mm_Horizontal
- moved D1 5.08 mm to (321.3, 169.9)
- moved D16 3.78 mm to (65.0, 131.1)
Routing:
- net Net-(D1-Pad1): track 858.3 -> 869.6 mm
- net Net-(D16-Pad2): track 15.7 -> 19.2 mm
- net Net-(CON1-Pad3): track 441.9 -> 443.1 mm
