File: hardware/kicad/cropdroid-room-v3/cropdroid-room.sch (KiCad schematic (older format))
At the start: 57 parts, among them CON1 SJ1-3523N, CON2 SJ1-3523N, CON3 SJ1-3523N, CON4 SJ1-3523N, CON5 SJ1-3523N, CON6 SJ1-3523N, CON7 SJ1-3523N, J1 703W-00_52, J2 3-213598-2, J3 3-213598-2, J4 3-213598-2, J5 3-213598-2, J6 3-213598-2, J7 3-213598-2, K1 T9AS1D12-15, K2 T9AS1D12-15, K3 T9AS1D12-15, K4 T9AS1D12-15, K5 T9AS1D12-15, K6 T9AS1D12-15, Q1 ULN2003AN, U1 IRM-30-12, U2 PPTC151LFBN-RC, U3 PPTC151LFBN-RC

Commit message: fix kicad v0.3a co2 circuit missing diode and connection to microcontroller
Parts:
- added D15: 1N4001, Diode_THT:D_DO-41_SOD81_P10.16mm_Horizontal, symbol Diode:1N4001
- renumbered D15 to D16, D16 to D17, D17 to D18, D18 to D19, D19 to D20, D20 to D21, D21 to D22, D22 to D23
Connections:
- net at U2.P$12: now also D15.1 (K)
- net at CON2.2 (T): now also D15.2 (A)
Changed lines of the file:
@@
 Title "CropDroid Room"
 Date "2020-02-03"
-Rev "v0.3a"
+Rev "v0.4a"
 Comp "Automate The Things, LLC"
 Comment1 ""
@@
 	12050 5900 12050 5050
 $Comp
-L Device:D_Photo D17
+L Device:D_Photo D18
 U 1 1 5E42A07B
 P 11750 5050
-F 0 "D17" H 11700 5345 50  0000 C CNN
+F 0 "D18" H 11700 5345 50  0000 C CNN
 F 1 "D_Photo" H 11700 5254 50  0000 C CNN
 F 2 "libraries:PHODET_PDV-P8103" H 11700 5050 50  0001 C CNN
@@
 	12050 2900 12050 3300
 $Comp
-L Diode:1N4001 D22
+L Diode:1N4001 D23
 U 1 1 5EB9F206
 P 13750 1850
-F 0 "D22" V 13796 1770 50  0000 R CNN
+F 0 "D23" V 13796 1770 50  0000 R CNN
 F 1 "1N4001" V 13705 1770 50  0000 R CNN
 F 2 "Diode_THT:D_DO-41_SOD81_P10.16mm_Horizontal" H 13750 1675 50  0001 C CNN
@@
 	13750 2000 13750 3300
 $Comp
-L Diode:1N4001 D20
+L Diode:1N4001 D21
 U 1 1 5EBA049F
 P 12700 1850
-F 0 "D20" V 12746 1770 50  0000 R CNN
+F 0 "D21" V 12746 1770 50  0000 R CNN
 F 1 "1N4001" V 12655 1770 50  0000 R CNN
 F 2 "Diode_THT:D_DO-41_SOD81_P10.16mm_Horizontal" H 12700 1675 50  0001 C CNN
@@
 	12700 2000 12700 3300
 $Comp
-L Diode:1N4001 D19
+L Diode:1N4001 D20
 U 1 1 5EBB6D0B
 P 12150 4400
-F 0 "D19" V 12196 4320 50  0000 R CNN
+F 0 "D20" V 12196 4320 50  0000 R CNN
 F 1 "1N4001" V 12105 4320 50  0000 R CNN
 F 2 "Diode_THT:D_DO-41_SOD81_P10.16mm_Horizontal" H 12150 4225 50  0001 C CNN
@@
 	12150 4550 12150 5900
 $Comp
-L Diode:1N4001 D21
+L Diode:1N4001 D22
 U 1 1 5EBB9A05
 P 13300 4400
-F 0 "D21" V 13346 4320 50  0000 R CNN
+F 0 "D22" V 13346 4320 50  0000 R CNN
 F 1 "1N4001" V 13255 4320 50  0000 R CNN
 F 2 "Diode_THT:D_DO-41_SOD81_P10.16mm_Horizontal" H 13300 4225 50  0001 C CNN
@@
 Wire Wire Line
 	3200 3550 3200 4150
-Wire Wire Line
-	9450 1600 9450 1750
-$Comp
-L Diode:1N4001 D18
+$Comp
+L Diode:1N4001 D19
 U 1 1 5EC94F68
 P 12050 3750
-F 0 "D18" V 12096 3670 50  0000 R CNN
+F 0 "D19" V 12096 3670 50  0000 R CNN
 F 1 "1N4001" V 12005 3670 50  0000 R CNN
 F 2 "Diode_THT:D_DO-41_SOD81_P10.16mm_Horizontal" H 12050 3575 50  0001 C CNN
@@
 	11450 1450 11450 1700
 $Comp
-L Diode:1N4001 D16
+L Diode:1N4001 D17
 U 1 1 5EBA0A16
 P 11450 1850
-F 0 "D16" V 11496 1770 50  0000 R CNN
+F 0 "D17" V 11496 1770 50  0000 R CNN
 F 1 "1N4001" V 11405 1770 50  0000 R CNN
 F 2 "Diode_THT:D_DO-41_SOD81_P10.16mm_Horizontal" H 11450 1675 50  0001 C CNN
@@
 	11000 1200 7850 1200
 $Comp
-L Diode:1N5400 D15
+L Diode:1N5400 D16
 U 1 1 5ECCD1A7
 P 11000 3300
-F 0 "D15" V 11046 3220 50  0000 R CNN
+F 0 "D16" V 11046 3220 50  0000 R CNN
 F 1 "1N5400" V 10955 3220 50  0000 R CNN
 F 2 "Diode_THT:D_DO-201AD_P15.24mm_Horizontal" H 11000 3125 50  0001 C CNN
@@
 Connection ~ 10400 8900
 Wire Wire Line
-	10500 1600 10500 9150
+	10500 1600 10500 8250
 $Comp
 L power:GND #PWR012
@@
 	9300 9150 9300 8900
 Connection ~ 9300 8900
+Wire Wire Line
+	10500 8550 10500 9150
+$Comp
+L Diode:1N4001 D15
+U 1 1 5E4770B0
+P 10500 8400
+F 0 "D15" V 10546 8320 50  0000 R CNN
+F 1 "1N4001" V 10455 8320 50  0000 R CNN
+F 2 "Diode_THT:D_DO-41_SOD81_P10.16mm_Horizontal" H 10500 8225 50  0001 C CNN
+F 3 "http://www.vishay.com/docs/88503/1n4001.pdf" H 10500 8400 50  0001 C CNN
+	1    10500 8400
+	0    1    1    0
+$EndComp
+Wire Wire Line
+	9450 1600 9450 1700
 $EndSCHEMATC

Commit message: more v0.3a fixes
Parts:
- removed D1: 1N4001, Diode_THT:D_DO-41_SOD81_P10.16mm_Horizontal, symbol Diode:1N4001
- removed D16: 1N5400, Diode_THT:D_DO-201AD_P15.24mm_Horizontal, symbol Diode:1N5400
- added D1: 1N5400, Diode_THT:D_DO-201AD_P15.24mm_Horizontal, symbol Diode:1N5400
- added D16: 1N4001, Diode_THT:D_DO-41_SOD81_P10.16mm_Horizontal, symbol Diode:1N4001
Connections:
- net at CON1.3 (R), CON2.3 (R), CON3.3 (R)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: now also D16.1 (K)
- net at D10.1 (K), D11.2 (A), D12.1 (K)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: now also D1.1 (K)
- net at U2.P$4: now also D16.2 (A)
- net at U1.4 (+V): now also D1.2 (A)
Changed lines of the file:
@@
 Wire Wire Line
 	13300 4550 13300 5900
-$Comp
-L Diode:1N4001 D1
-U 1 1 5EBC673C
-P 3200 3400
-F 0 "D1" V 3246 3320 50  0000 R CNN
-F 1 "1N4001" V 3155 3320 50  0000 R CNN
-F 2 "Diode_THT:D_DO-41_SOD81_P10.16mm_Horizontal" H 3200 3225 50  0001 C CNN
-F 3 "http://www.vishay.com/docs/88503/1n4001.pdf" H 3200 3400 50  0001 C CNN
-	1    3200 3400
-	0    -1   -1   0
-$EndComp
 Wire Wire Line
 	3200 3550 3200 4150
@@
 Wire Wire Line
 	11000 1200 11000 3150
-Connection ~ 11000 3450
 $Comp
 L power:GND #PWR013
@@
 Wire Wire Line
 	11000 1200 7850 1200
-$Comp
-L Diode:1N5400 D16
-U 1 1 5ECCD1A7
-P 11000 3300
-F 0 "D16" V 11046 3220 50  0000 R CNN
-F 1 "1N5400" V 10955 3220 50  0000 R CNN
-F 2 "Diode_THT:D_DO-201AD_P15.24mm_Horizontal" H 11000 3125 50  0001 C CNN
-F 3 "http://www.vishay.com/docs/88516/1n5400.pdf" H 11000 3300 50  0001 C CNN
-	1    11000 3300
-	0    -1   -1   0
-$EndComp
 $Comp
 L Device:R R8
@@
 Wire Wire Line
 	9450 1600 9450 1700
+$Comp
+L Diode:1N5400 D1
+U 1 1 5E4BA390
+P 3200 3400
+F 0 "D1" V 3246 3320 50  0000 R CNN
+F 1 "1N5400" V 3155 3320 50  0000 R CNN
+F 2 "Diode_THT:D_DO-201AD_P15.24mm_Horizontal" H 3200 3225 50  0001 C CNN
+F 3 "http://www.vishay.com/docs/88516/1n5400.pdf" H 3200 3400 50  0001 C CNN
+	1    3200 3400
+	0    -1   -1   0
+$EndComp
+$Comp
+L Diode:1N4001 D16
+U 1 1 5E4CF1FB
+P 11000 3300
+F 0 "D16" V 11046 3220 50  0000 R CNN
+F 1 "1N4001" V 10955 3220 50  0000 R CNN
+F 2 "Diode_THT:D_DO-41_SOD81_P10.16mm_Horizontal" H 11000 3125 50  0001 C CNN
+F 3 "http://www.vishay.com/docs/88503/1n4001.pdf" H 11000 3300 50  0001 C CNN
+	1    11000 3300
+	0    -1   -1   0
+$EndComp
+Connection ~ 11000 3450
 $EndSCHEMATC
