File: hardware/kicad/cropdroid-room-v0.4a/cropdroid-room.kicad_pcb (KiCad board)
At the start: 2 copper layers, 377.2 x 131.1 mm, 63 parts, among them CON1 SJ1-3523N, CON2 SJ1-3523N, CON3 SJ1-3523N, CON4 SJ1-3523N, CON5 SJ1-3523N, CON6 SJ1-3523N, CON7 SJ1-3523N, J1 703W-00_52, J2 3-213598-2, J3 3-213598-2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

Commit message: room v0.4a
Parts:
- removed D1: 1N5400, Diode_THT:D_DO-201AD_P15.24mm_Horizontal
- removed D17: 1N4001, Diode_THT:D_DO-41_SOD81_P10.16mm_Horizontal
Connections:
- D10 pad 1: Net-(D1-Pad1) -> Net-(D10-Pad1)
- D11 pad 2: Net-(D1-Pad1) -> Net-(D10-Pad1)
- D12 pad 1: Net-(D1-Pad1) -> Net-(D10-Pad1)
- D13 pad 2: Net-(D1-Pad1) -> Net-(D10-Pad1)
- D18 pad 1: Net-(D17-Pad2) -> Net-(D18-Pad1)
- D2 pad 1: Net-(D1-Pad1) -> Net-(D10-Pad1)
- D3 pad 2: Net-(D1-Pad1) -> Net-(D10-Pad1)
- D4 pad 1: Net-(D1-Pad1) -> Net-(D10-Pad1)
- D5 pad 2: Net-(D1-Pad1) -> Net-(D10-Pad1)
- D6 pad 1: Net-(D1-Pad1) -> Net-(D10-Pad1)
- D7 pad 2: Net-(D1-Pad1) -> Net-(D10-Pad1)
- D8 pad 1: Net-(D1-Pad1) -> Net-(D10-Pad1)
- D9 pad 2: Net-(D1-Pad1) -> Net-(D10-Pad1)
- K1 pad 2: Net-(D1-Pad1) -> Net-(D10-Pad1)
- K2 pad 2: Net-(D1-Pad1) -> Net-(D10-Pad1)
- K3 pad 2: Net-(D1-Pad1) -> Net-(D10-Pad1)
- K4 pad 2: Net-(D1-Pad1) -> Net-(D10-Pad1)
- K5 pad 2: Net-(D1-Pad1) -> Net-(D10-Pad1)
- K6 pad 2: Net-(D1-Pad1) -> Net-(D10-Pad1)
- Q1 pad 9: Net-(D1-Pad1) -> Net-(D10-Pad1)
- R8 pad 1: Net-(D17-Pad2) -> Net-(D18-Pad1)
- U1 pad 4: Net-(D1-Pad2) -> Net-(D10-Pad1)
- U2 pad P$1: Net-(D1-Pad1) -> Net-(D10-Pad1)
- U2 pad P$9: Net-(D17-Pad1) -> Net-(D18-Pad1)
Routing:
- net Net-(D10-Pad1): track 0.00 -> 878.0 mm
- net Net-(D1-Pad1): track 869.6 -> 0.00 mm
- net Net-(D18-Pad1): track 0.00 -> 75.6 mm
- net Net-(D17-Pad1): track 54.4 -> 0.00 mm
- net Net-(D1-Pad2): track 35.5 -> 0.00 mm
- net Net-(D17-Pad2): track 11.8 -> 0.00 mm
Other:
- board text added: "CropDroid Room Controller CopyRight (c) Automate The Things, LLC Prototype v0.4a"
- board text removed: "CropDroid Room Controller CopyRight (c) Automate The Things, LLC Prototype v0.3a"

Commit message: add v0.5a hardware
Parts:
- removed the Screw at (29.0, 119.4)
- removed the Screw at (388.1, 169.9)
- removed the Screw at (104.9, 58.9)
- removed the Screw at (354.1, 86.6)
- added Screw: Drill, drill-hole:Drill_Hole, F.Cu at (390.5, 168.0)
- added Screw: Drill, drill-hole:Drill_Hole, F.Cu at (353.2, 86.2)
- added Screw: Drill, drill-hole:Drill_Hole, F.Cu at (103.3, 65.3)
- added Screw: Drill, drill-hole:Drill_Hole, F.Cu at (40.0, 123.3)
